File: pcb/Reflow-Controller-Kicad/Reflow-Controller-Kicad.kicad_sch (KiCad schematic)
At the start: 61 parts, among them J1 , J10 , J2 USB_C_Receptacle_USB2.0, J3 , J4 , J5 , J6 , J7 , J8 , J9 Servo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

Commit message: Update
Parts:
- added J11: Conn_01x08, footprint:0.96_TFT_Display_ST77335S, symbol Connector_Generic:Conn_01x08
- added JP3, JP4: (no value), Jumper:SolderJumper-3_P2.0mm_Open_TrianglePad1.0x1.5mm, symbol Jumper:SolderJumper_3_Open
Connections:
- net +3.3V: now also J11.2 (Pin_2), J11.8 (Pin_8), JP3.3 (B); no longer J10.2 (Pin_2)
- net CLK: now also JP4.1 (A)
- net GND: now also J11.1 (Pin_1), JP4.3 (B); no longer J10.1 (Pin_1)
- net MOSI: now also JP3.1 (A)
- net SCL: now also J11.5 (Pin_5)
- net SDA: now also J11.6 (Pin_6)
- net CS_DISPLAY: now reaches U1.30 (IO36)
- net CS_DISPLAY: now also J11.7 (Pin_7)
- new net: J10.2 (Pin_2), J11.4 (Pin_4), JP3.2 (C)
- new net: J10.1 (Pin_1), J11.3 (Pin_3), JP4.2 (C)
Other:
- moved on the sheet: H1, H2, H3, H4, J10, R12, R13, R14
